File: solder_station_board.sch (KiCad schematic (older format))
At the start: 43 parts, among them J1 PWR_5_V, J2 INPUT, J3 RT_WELLER, J4 INPUT, J5 VFD_DISPLAY, J6 PWR_15V, J8 SERIAL, P1 ISP, Q1 IRF9540, Q2 2N7002, U4 TLC272, U5 LT1007, U6 ATMEGA168-20AU

Commit message: remove 0R resistors
Parts:
- removed R1, R2: 0, Resistor_SMD:R_1206_3216Metric, symbol Device:R_Small
Changed lines of the file:
@@
 EESchema Schematic File Version 4
 LIBS:solder_station_board-cache
-EELAYER 29 0
+EELAYER 26 0
 EELAYER END
 $Descr A4 11693 8268
@@
 	1    0    0    -1
 $EndComp
-$Comp
-L power:+5V #PWR04
-U 1 1 5CB070E5
-P 8650 5800
-F 0 "#PWR04" H 8650 5650 50  0001 C CNN
-F 1 "+5V" H 8665 5973 50  0000 C CNN
-F 2 "" H 8650 5800 50  0001 C CNN
-F 3 "" H 8650 5800 50  0001 C CNN
-	1    8650 5800
-	1    0    0    -1
-$EndComp
-$Comp
-L Device:R_Small R1
-U 1 1 5CB07375
-P 8850 5900
-F 0 "R1" V 8654 5900 50  0000 C CNN
-F 1 "0" V 8745 5900 50  0000 C CNN
-F 2 "Resistor_SMD:R_1206_3216Metric" H 8850 5900 50  0001 C CNN
-F 3 "~" H 8850 5900 50  0001 C CNN
-	1    8850 5900
-	0    1    1    0
-$EndComp
-$Comp
-L power:+5V #PWR05
-U 1 1 5CB074F4
-P 9050 5800
-F 0 "#PWR05" H 9050 5650 50  0001 C CNN
-F 1 "+5V" H 9065 5973 50  0000 C CNN
-F 2 "" H 9050 5800 50  0001 C CNN
-F 3 "" H 9050 5800 50  0001 C CNN
-	1    9050 5800
-	1    0    0    -1
-$EndComp
-Wire Wire Line
-	9050 5800 9050 5900
-Wire Wire Line
-	9050 5900 8950 5900
-Wire Wire Line
-	8750 5900 8650 5900
-Wire Wire Line
-	8650 5900 8650 5800
-$Comp
-L Device:R_Small R2
-U 1 1 5CB13331
-P 8850 6100
-F 0 "R2" V 8654 6100 50  0000 C CNN
-F 1 "0" V 8745 6100 50  0000 C CNN
-F 2 "Resistor_SMD:R_1206_3216Metric" H 8850 6100 50  0001 C CNN
-F 3 "~" H 8850 6100 50  0001 C CNN
-	1    8850 6100
-	0    1    1    0
-$EndComp
-Wire Wire Line
-	8950 6100 9050 6100
-Wire Wire Line
-	9050 6100 9050 5900
-Connection ~ 9050 5900
-Wire Wire Line
-	8650 5900 8650 6100
-Wire Wire Line
-	8650 6100 8750 6100
-Connection ~ 8650 5900
 $EndSCHEMATC

Commit message: small arrangements
Parts:
- removed C1, C13, C2: 10n, Capacitor_SMD:C_0805_2012Metric_Pad1.15x1.40mm_HandSolder, symbol Device:C_Small
- removed J1: PWR_5_V, Connector_PinSocket_2.54mm:PinSocket_1x03_P2.54mm_Vertical, symbol Connector_Generic:Conn_01x03
- removed J2: INPUT, Connector_PinHeader_2.54mm:PinHeader_1x04_P2.54mm_Vertical, symbol Connector_Generic:Conn_01x04
- removed R13, R16, R4: 1k, Resistor_SMD:R_0805_2012Metric_Pad1.15x1.40mm_HandSolder, symbol Device:R_Small
- removed R14: 33k, Resistor_SMD:R_0805_2012Metric_Pad1.15x1.40mm_HandSolder, symbol Device:R_Small
- removed R15: 10K, Resistor_SMD:R_0805_2012Metric_Pad1.15x1.40mm_HandSolder, symbol Device:R_Small
- removed TP1, TP2, TP3: tp, Connector_Wire:SolderWirePad_1x01_Drill0.8mm, symbol solder_station_board-rescue:TestPoint-Connector
- removed U4: TLC272, Package_SO:SOIC-8_3.9x4.9mm_P1.27mm, symbol Amplifier_Operational:TLC272
- removed U5: LT1007, Package_SO:SOIC-8_3.9x4.9mm_P1.27mm, symbol Amplifier_Operational:LT1012
- added C4: 10n, Capacitor_SMD:C_0805_2012Metric_Pad1.15x1.40mm_HandSolder, symbol Device:C_Small
- added C5, C7: 100n, Capacitor_SMD:C_0805_2012Metric_Pad1.15x1.40mm_HandSolder, symbol Device:C_Small
- added C6: 100u, Capacitor_THT:C_Radial_D8.0mm_H7.0mm_P3.50mm, symbol Device:CP_Small
- added D3: LED_G, LED_THT:LED_D3.0mm, symbol solder_station_board-rescue:LED_Small-custom
- added J4: PWR_5V, Connector_PinHeader_2.54mm:PinHeader_1x02_P2.54mm_Vertical, symbol Connector_Generic:Conn_01x02
- added J6: ENCODER, Connector_PinHeader_2.54mm:PinHeader_1x05_P2.54mm_Vertical, symbol Connector_Generic:Conn_01x05
- added L1: 10u, Inductor_SMD:L_1206_3216Metric_Pad1.42x1.75mm_HandSolder, symbol Device:L_Small
- added R1: 10M, Resistor_SMD:R_0805_2012Metric_Pad1.15x1.40mm_HandSolder, symbol Device:R_Small
- added R11: 1k, Resistor_SMD:R_0805_2012Metric_Pad1.15x1.40mm_HandSolder, symbol Device:R_Small
- added R5: 68k, Resistor_SMD:R_0805_2012Metric_Pad1.15x1.40mm_HandSolder, symbol Device:R_Small
- added R7: 5k6, Resistor_SMD:R_0805_2012Metric_Pad1.15x1.40mm_HandSolder, symbol Device:R_Small
- added TP1: TEMP, TestPoint:TestPoint_Loop_D2.60mm_Drill0.9mm_Beaded, symbol Connector:TestPoint
- added U1: OPA343, Package_TO_SOT_SMD:SOT-23-5, symbol Amplifier_Operational:OPA340NA
- MH1, MH2, MH3, MH4: value MountingHole_Pad -> MH_Pad
- R12: value 22k -> 648
- R6: renamed from R10; value 1k -> 100
- renumbered C7 to C1, C8 to C2, C9 to C3, D8 to D2, J3 to J1, J8 to J2, J6 to J3, J4 to J7, R6 to R10, R5 to R2, R7 to R3, R11 to R4, R9 to R8, R8 to R9, U6 to U2
Connections:
- net +5V: now also R12.2, C6.1, J4.2 (Pin_2), J6.4 (Pin_4), L1.1, R1.2, R11.1, U1.5 (V+); no longer U2.18 (AVCC)
- net GND: now also R6.2, C4.2, C5.2, C6.2, C7.2, D3.1 (K), J4.1 (Pin_1), J6.5 (Pin_5), U1.2 (V-)
- net INP1: now also J6.1 (Pin_1)
- net INP2: now also J6.2 (Pin_2)
- net INP3: now also J6.3 (Pin_3)
- net RST: now also C5.1, R11.2
- net TEMP: now also C4.1, R7.1, TP1.1
- net at J1.1 (Pin_1), R2.2: now also R1.1
- net at C1.1, R2.1, R3.2: now also U1.3 (+)
- net at R12.1: now also D3.2 (A); no longer R6.2
- net at R6.1: now also R5.2, U1.4 (-)
- net RX: now reaches J2.1 (Pin_1), U2.30 ((PCINT16/RXD)PD0)
- net TX: now reaches J2.2 (Pin_2), U2.31 ((PCINT17/TXD)PD1)
- new net: C7.1, L1.2, U2.18 (AVCC)
- new net: R5.1, R7.2, U1.1
- no-connect marks 15 -> 12
Other:
- moved on the sheet: C1, C2, C3, D1, D2, J1, J2, J3, J5, J7, MH1, MH2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

Commit message: two rt_weller
Parts:
- removed D1: BAT54S, Package_TO_SOT_SMD:SOT-23, symbol Diode:BAT54S
- removed D3: LED_G, LED_THT:LED_D3.0mm, symbol solder_station_board-rescue:LED_Small-custom
- removed U1: OPA343, Package_TO_SOT_SMD:SOT-23-5, symbol Amplifier_Operational:OPA340NA
- added C10: 10n, Capacitor_SMD:C_0805_2012Metric_Pad1.15x1.40mm_HandSolder, symbol Device:C_Small
- added C8: 100n, Capacitor_SMD:C_0805_2012Metric_Pad1.15x1.40mm_HandSolder, symbol Device:C_Small
- added C9: 8n2, Capacitor_SMD:C_0805_2012Metric_Pad1.15x1.40mm_HandSolder, symbol Device:C_Small
- added D1: LED_G, LED_THT:LED_D3.0mm, symbol Device:LED_Small
- added J10: OW_DISPLAY, Connector_PinHeader_2.54mm:PinHeader_1x04_P2.54mm_Vertical, symbol Connector_Generic:Conn_01x04
- added J8: PORT, Connector_PinHeader_2.54mm:PinHeader_1x05_P2.54mm_Vertical, symbol Connector_Generic:Conn_01x05
- added J9: RT_WELLER, Connector_PinSocket_2.54mm:PinSocket_1x03_P2.54mm_Vertical, symbol Connector_Generic:Conn_01x03
- added Q3: IRLM6401, Package_TO_SOT_SMD:SOT-23, symbol Device:Q_PMOS_GSD
- added Q4: IRF9540, Package_TO_SOT_THT:TO-220-3_Vertical, symbol Device:Q_PMOS_GDS
- added Q5: 2N7002, Package_TO_SOT_SMD:SOT-23, symbol Transistor_FET:2N7002
- added R13: 1k, Resistor_SMD:R_0805_2012Metric_Pad1.15x1.40mm_HandSolder, symbol Device:R_Small
- added R14: 100K, Resistor_SMD:R_0805_2012Metric_Pad1.15x1.40mm_HandSolder, symbol Device:R_Small
- added R15: 2k2, Resistor_SMD:R_0805_2012Metric_Pad1.15x1.40mm_HandSolder, symbol Device:R_Small
- added R16: 4k7, Resistor_SMD:R_0805_2012Metric_Pad1.15x1.40mm_HandSolder, symbol Device:R_Small
- added R17: 10M, Resistor_SMD:R_0805_2012Metric_Pad1.15x1.40mm_HandSolder, symbol Device:R_Small
- added R18, R22: 5k6, Resistor_SMD:R_0805_2012Metric_Pad1.15x1.40mm_HandSolder, symbol Device:R_Small
- added R19: 100k, Resistor_SMD:R_0805_2012Metric_Pad1.15x1.40mm_HandSolder, symbol Device:R_Small
- added R20: 39k, Resistor_SMD:R_0805_2012Metric_Pad1.15x1.40mm_HandSolder, symbol Device:R_Small
- added R21: 100, Resistor_SMD:R_0805_2012Metric_Pad1.15x1.40mm_HandSolder, symbol Device:R_Small
- added TP2: TEMP, TestPoint:TestPoint_Loop_D2.60mm_Drill0.9mm_Beaded, symbol Connector:TestPoint
- added U1: OPA2343, Package_SO:SOIC-8_3.9x4.9mm_P1.27mm, symbol Amplifier_Operational:OPA2340
- C1: value 10n -> 8n2
- D2: footprint Diode_SMD:D_MicroMELF_Hadsoldering -> Diode_SMD:D_1206_3216Metric_Castellated
- J6: footprint Connector_PinHeader_2.54mm:PinHeader_1x05_P2.54mm_Vertical -> Connector_PinHeader_2.54mm:PinHeader_1x04_P2.54mm_Vertical; symbol Connector_Generic:Conn_01x05 -> Connector_Generic:Conn_01x04
- J7: value INPUT -> PORTB
- Q1: footprint Package_TO_SOT_THT:TO-220-3_Horizontal_TabDown -> Package_TO_SOT_THT:TO-220-3_Vertical
- R4: value 1k -> 560
- R5: value 68k -> 39k
Connections:
- net +15V: now also Q4.3 (S), R16.1
- net +5V: now also C8.1, J10.4 (Pin_4), Q3.2 (S), R17.2, U1.8 (V+); no longer J4.2 (Pin_2)
- net GND: now also J2.1 (Pin_1), J5.1 (Pin_1), J6.1 (Pin_1), J7.1 (Pin_1), C10.2, C8.2, C9.2, D1.1 (K), J10.1 (Pin_1), J8.1 (Pin_1), J9.3 (Pin_3), Q5.2 (S), R14.1, R15.1, R19.1, R21.2, U1.4 (V-); no longer J2.3 (Pin_3), J5.5 (Pin_5), J6.5 (Pin_5), J7.4 (Pin_4)
- net RX: now also J2.3 (Pin_3); no longer J2.1 (Pin_1)
- net VFD_DATA: now also J5.5 (Pin_5), U2.28 ((PCINT13/SCL/ADC5)PC5); no longer J5.1 (Pin_1), U2.27 ((PCINT12/SDA/ADC4)PC4)
- net VFD_RCLK: now also J5.4 (Pin_4), U2.27 ((PCINT12/SDA/ADC4)PC4); no longer J5.2 (Pin_2), U2.26 ((PCINT11/ADC3)PC3)
- net VFD_SRCLK: now also U2.26 ((PCINT11/ADC3)PC3); no longer U2.25 ((PCINT10/ADC2)PC2)
- net ~VFD_SRCLR: now also J5.2 (Pin_2), U2.25 ((PCINT10/ADC2)PC2); no longer J5.4 (Pin_4), U2.24 ((PCINT9/ADC1)PC1)
- net HEAT_H: now reaches Q1.2 (D)
- net HEAT_H: now also J9.2 (Pin_2); no longer J1.2 (Pin_2)
- net at C1.1, R2.1, R3.2: now also U1.3 (+)
- net at R5.2, R6.1: now also U1.2 (-)
- net PB1: now reaches U2.12 ((PCINT0/CLKO/ICP1)PB0)
- net PB1: now also J7.4 (Pin_4)
- net SOLDER_H: now reaches U2.13 ((PCINT1/OC1A)PB1)
- net SOLDER_H: now also R8.1
- net SOLDER_L: now reaches U2.14 ((PCINT2/OC1B/~SS~)PB2)
- net SOLDER_L: now also R13.1
- net TEMP_H: now reaches U2.22 (ADC7)
- net TEMP_H: now also C10.1, R22.1, TP2.1
- net PB6: now reaches U2.7 ((PCINT6/XTAL1/TOSC1)PB6)
- net PB6: now also J7.3 (Pin_3)
- net PB7: now reaches U2.8 ((PCINT7/XTAL2/TOSC2)PB7)
- net PB7: now also J7.2 (Pin_2)
- net at R5.1, R7.2: now also U1.1
- net at R12.1: now also D1.2 (A)
- net INP1 renamed PD2
- net PD2: now also J8.3 (Pin_3); no longer J6.1 (Pin_1)
- net INP2 renamed ENC_B
- net ENC_B: now also U2.2 ((PCINT20/XCK/T0)PD4); no longer U2.1 ((PCINT19/OC2B/INT1)PD3)
- net INP3 renamed ENC_A
- net ENC_A: now also U2.9 ((PCINT21/OC0B/T1)PD5); no longer U2.2 ((PCINT20/XCK/T0)PD4)
- removed net INP4: J7.1 (Pin_1), U2.9 ((PCINT21/OC0B/T1)PD5)
- net INP5 renamed OW_DIO
- net OW_DIO: now also J10.3 (Pin_3); no longer J7.2 (Pin_2)
- net INP6 renamed OW_RST
- net OW_RST: now also J10.2 (Pin_2); no longer J7.3 (Pin_3)
- net SOLDER renamed PC0
- net PC0: now also J8.5 (Pin_5); no longer R8.1
- net TEMP renamed TEMP_L
- new net: J4.2 (Pin_2), Q3.3 (D)
- new net: Q4.1 (G), Q5.3 (D), R16.2
- new net: Q5.1 (G), R13.2, R15.2
- new net: J9.1 (Pin_1), R17.1, R18.2
- new net: C9.1, R18.1, R19.2, U1.5 (+)
- new net: R20.2, R21.1, U1.6 (-)
- new net: R20.1, R22.2, U1.7
- new net: Q3.1 (G), R14.2
- new net HEAT_L: J1.2 (Pin_2), Q4.2 (D)
- new net PC1: J8.4 (Pin_4), U2.24 ((PCINT9/ADC1)PC1)
- new net PD3: J8.2 (Pin_2), U2.1 ((PCINT19/OC2B/INT1)PD3)
- no-connect marks 12 -> 5
Other:
- moved on the sheet: C1, C4, J1, J2, J3, J4, J5, J7, P1, Q1, Q2, R1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
